File: electronic_load.kicad_sch (KiCad schematic)
At the start: 49 parts, among them J1 Conn_01x02, J2 Conn_01x03, J3 Conn_01x03_Pin, J4 Conn_01x06_Pin, J5 Conn_01x04_Pin, J6 Conn_01x14_Pin, J7 USB_C_Receptacle_USB2.0_16P, U1 STM32G491METx, U3 MCP4728, U4 LF33_TO252, U5 NCP1117-5.0_SOT223, U6 USBLC6-2SC6, Y1 12MHz

Commit message: changing the operational amplifier
Parts:
- J1: footprint (none) -> Connector_BarrelJack:BarrelJack_Wuerth_694108106102_2.5x5.5mm
- J2: footprint (none) -> Connector_Samtec_HPM_THT:Samtec_HPM-03-01-x-S_Straight_1x03_Pitch5.08mm
- J3: footprint (none) -> Connector_PinSocket_2.54mm:PinSocket_1x03_P2.54mm_Vertical
- J4: footprint (none) -> Connector_PinSocket_2.54mm:PinSocket_1x06_P2.54mm_Vertical
- J5: footprint (none) -> Connector_PinSocket_2.54mm:PinSocket_1x04_P2.54mm_Vertical
- J6: footprint (none) -> Connector_PinSocket_2.54mm:PinSocket_1x14_P2.54mm_Vertical
- J7: footprint (none) -> Connector_USB:USB_C_Receptacle_GCT_USB4105-xx-A_16P_TopMnt_Horizontal
- renumbered U3 to U2, U4 to U3, U5 to U4, U6 to U5
Connections:
- net DAC_LDAC: now also U1.53 (PC7); no longer U1.75 (PB6)
- net DAC_RDY: now also U1.52 (PC6); no longer U1.74 (PB5)
- net DAC_SCL: now also U1.54 (PC8); no longer U1.77 (PB8)
- net DAC_SDA: now also U1.55 (PC9); no longer U1.76 (PB7)
- net DOWN: now also U1.74 (PB5); no longer U1.53 (PC7)
- net LEFT: now also U1.75 (PB6); no longer U1.54 (PC8)
- net OK: now also U1.72 (PB3); no longer U1.56 (PA8)
- net RIGHT: now also U1.76 (PB7); no longer U1.55 (PC9)
- net UP: now also U1.73 (PB4); no longer U1.52 (PC6)
- net USB_DM: now also U5.6 (I/O1); no longer U5.4 (I/O2)
- net USB_DP: now also U5.4 (I/O2); no longer U5.6 (I/O1)
- net at J7.A6 (D+), J7.B6 (D+): now also U5.3 (I/O2); no longer U5.1 (I/O1)
- net at J7.A7 (D-), J7.B7 (D-): now also U5.1 (I/O1); no longer U5.3 (I/O2)
Other:
- moved on the sheet: U5

Commit message: connectors
Parts:
- removed J1: Conn_01x02, Connector_BarrelJack:BarrelJack_Wuerth_694108106102_2.5x5.5mm, symbol Connector_Generic:Conn_01x02
- added J1: Barrel_Jack_Switch_Pin3Ring, Connector_BarrelJack:BarrelJack_Wuerth_694106106102_2.0x5.5mm, symbol Connector:Barrel_Jack_Switch_Pin3Ring
Connections:
- net +12V: now also J1.1
- net GND: now also J1.2
- no-connect marks 27 -> 28
Changed lines of the file:
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@@
 	)
 	(no_connect
+		(at 21.59 20.32)
+	)
+	(no_connect
 		(at 222.25 106.68)
 	)
@@
 	(wire
 		(pts
-			(xy 21.59 22.86) (xy 20.32 22.86)
-		)
-		(stroke
-			(width 0)
-			(type default)
-		)
-	)
-	(wire
-		(pts
 			(xy 35.56 187.96) (xy 35.56 186.69)
 		)
@@
 	(wire
 		(pts
+			(xy 21.59 25.4) (xy 17.78 25.4)
+		)
+		(stroke
+			(width 0)
+			(type default)
+		)
+	)
+	(wire
+		(pts
 			(xy 113.03 49.53) (xy 113.03 52.07)
 		)
@@
 	(wire
 		(pts
+			(xy 20.32 22.86) (xy 21.59 22.86)
+		)
+		(stroke
+			(width 0)
+			(type default)
+		)
+	)
+	(wire
+		(pts
 			(xy 128.27 184.15) (xy 132.08 184.15)
 		)
@@
 	(wire
 		(pts
-			(xy 20.32 25.4) (xy 20.32 29.21)
-		)
-		(stroke
-			(width 0)
-			(type default)
-		)
-	)
-	(wire
-		(pts
 			(xy 27.94 93.98) (xy 44.45 93.98)
 		)
@@
 	(wire
 		(pts
-			(xy 21.59 25.4) (xy 20.32 25.4)
-		)
-		(stroke
-			(width 0)
-			(type default)
-		)
-	)
-	(wire
-		(pts
 			(xy 262.89 114.3) (xy 266.7 114.3)
 		)
@@
 	(wire
 		(pts
-			(xy 20.32 22.86) (xy 20.32 19.05)
+			(xy 17.78 19.05) (xy 17.78 25.4)
 		)
 		(stroke
@@
 	(wire
 		(pts
+			(xy 20.32 29.21) (xy 20.32 22.86)
+		)
+		(stroke
+			(width 0)
+			(type default)
+		)
+	)
+	(wire
+		(pts
 			(xy 218.44 124.46) (xy 222.25 124.46)
 		)
@@
 	)
 	(symbol
-		(lib_id "Connector_Generic:Conn_01x02")
-		(at 26.67 22.86 0)
-		(unit 1)
-		(body_style 1)
-		(exclude_from_sim no)
-		(in_bom yes)
-		(on_board yes)
-		(in_pos_files yes)
-		(dnp no)
-		(fields_autoplaced yes)
-		(property "Reference" "J1"
-			(at 29.21 24.1299 0)
-			(show_name no)
-			(do_not_autoplace no)
-			(effects
-				(font
-					(size 1.27 1.27)
-				)
-				(justify left)
-			)
-		)
-		(property "Value" "Conn_01x02"
-			(at 29.21 25.3999 0)
-			(hide yes)
-			(show_name no)
-			(do_not_autoplace no)
-			(effects
-				(font
-					(size 1.27 1.27)
-				)
-				(justify left)
-			)
-		)
-		(property "Footprint" "Connector_BarrelJack:BarrelJack_Wuerth_694108106102_2.5x5.5mm"
-			(at 26.67 22.86 0)
-			(hide yes)
-			(show_name no)
-			(do_not_autoplace no)
-			(effects
-				(font
-					(size 1.27 1.27)
-				)
-			)
-		)
-		(property "Datasheet" ""
-			(at 26.67 22.86 0)
-			(hide yes)
-			(show_name no)
-			(do_not_autoplace no)
-			(effects
-				(font
-					(size 1.27 1.27)
-				)
-			)
-		)
-		(property "Description" "Generic connector, single row, 01x02, script generated (kicad-library-utils/schlib/autogen/connector/)"
-			(at 26.67 22.86 0)
-			(hide yes)
-			(show_name no)
-			(do_not_autoplace no)
-			(effects
-				(font
-					(size 1.27 1.27)
-				)
-			)
-		)
-		(pin "1"
-		)
-		(pin "2"
-		)
-		(instances
-			(project "electronic_load"
-				(path "/eb6f2439-c99a-400f-b3b0-2a7303f23577"
-					(reference "J1")
-					(unit 1)
-				)
-			)
-		)
-	)
-	(symbol
 		(lib_id "Device:C_Small")
 		(at 106.68 57.15 0)
@@
 	(symbol
 		(lib_id "power:+12V")
-		(at 20.32 19.05 0)
+		(at 17.78 19.05 0)
 		(unit 1)
 		(body_style 1)
@@
 		(fields_autoplaced yes)
 		(property "Reference" "#PWR033"
-			(at 20.32 22.86 0)
+			(at 17.78 22.86 0)
 			(hide yes)
 			(show_name no)
@@
 		)
 		(property "Value" "+12V"
-			(at 20.32 15.24 0)
+			(at 17.78 15.24 0)
 			(show_name no)
 			(do_not_autoplace no)
@@
 		)
 		(property "Footprint" ""
-			(at 20.32 19.05 0)
+			(at 17.78 19.05 0)
 			(hide yes)
 			(show_name no)
@@
 		)
 		(property "Datasheet" ""
-			(at 20.32 19.05 0)
+			(at 17.78 19.05 0)
 			(hide yes)
 			(show_name no)
@@
 		)
 		(property "Description" "Power symbol creates a global label with name \"+12V\""
-			(at 20.32 19.05 0)
+			(at 17.78 19.05 0)
 			(hide yes)
 			(show_name no)
@@
 					(unit 1)
 				)
+			)
+		)
+	)
+	(symbol
+		(lib_id "Connector:Barrel_Jack_Switch_Pin3Ring")
+		(at 29.21 22.86 180)
+		(unit 1)
+		(body_style 1)
+		(exclude_from_sim no)
+		(in_bom yes)
+		(on_board yes)
+		(in_pos_files yes)
+		(dnp no)
+		(fields_autoplaced yes)
+		(property "Reference" "J1"
+			(at 35.56 21.5899 0)
+			(show_name no)
+			(do_not_autoplace no)
+			(effects
+				(font
+					(size 1.27 1.27)
+				)
+				(justify right)
+			)
+		)
+		(property "Value" "Barrel_Jack_Switch_Pin3Ring"
+			(at 35.56 24.1299 0)
+			(hide yes)
+			(show_name no)
+			(do_not_autoplace no)
+			(effects
+				(font
+					(size 1.27 1.27)
+				)
+				(justify right)
+			)
+		)
+		(property "Footprint" "Connector_BarrelJack:BarrelJack_Wuerth_694106106102_2.0x5.5mm"
+			(at 27.94 21.844 0)
+			(hide yes)
+			(show_name no)
+			(do_not_autoplace no)
+			(effects
+				(font
+					(size 1.27 1.27)
+				)
+			)
+		)
+		(property "Datasheet" ""
+			(at 27.94 21.844 0)
+			(hide yes)
+			(show_name no)
+			(do_not_autoplace no)
+			(effects
+				(font
+					(size 1.27 1.27)
+				)
+			)
+		)
+		(property "Description" "DC Barrel Jack with an internal switch"
+			(at 29.21 22.86 0)
+			(hide yes)
+			(show_name no)
+			(do_not_autoplace no)
+			(effects
+				(font
+					(size 1.27 1.27)
+				)
+			)
+		)
+		(pin "3"
+		)
+		(pin "2"
+		)
+		(pin "1"
+		)
+		(instances
+			(project "electronic_load"
+				(path "/eb6f2439-c99a-400f-b3b0-2a7303f23577"
+					(reference "J1")
+					(unit 1)
+				)

Commit message: connectors
Parts:
- removed J6: Conn_01x14_Pin, Connector_PinSocket_2.54mm:PinSocket_1x14_P2.54mm_Vertical, symbol Connector:Conn_01x14_Pin
- added J6: Conn_02x07_Top_Bottom, Connector_PinSocket_2.54mm:PinSocket_2x07_P2.54mm_Vertical, symbol Connector_Generic:Conn_02x07_Top_Bottom
Connections:
- net +3.3V: now also J6.1 (Pin_1), J6.8 (Pin_8)
- net CS: now also U1.49 (PD10), J6.3 (Pin_3); no longer U1.47 (PD8)
- net DC/RS: now also U1.47 (PD8), J6.5 (Pin_5); no longer U1.49 (PD10)
- net Fan1_PWM: now also U1.25 (PB1); no longer U1.24 (PB0)
- net Fan2_PWM: now also U1.24 (PB0); no longer U1.25 (PB1)
- net GND: now also J6.2 (Pin_2)
- net R1: now also U1.20 (PA6); no longer U1.17 (PA3)
- net R2: now also U1.19 (PA5); no longer U1.18 (PA4)
- net R3: now also U1.18 (PA4); no longer U1.19 (PA5)
- net R4: now also U1.17 (PA3); no longer U1.20 (PA6)
- net RESET: now also J6.4 (Pin_4)
- net SCK: now also J6.10 (Pin_10), J6.7 (Pin_7)
- net SDI(MOSI): now also J6.12 (Pin_12), J6.6 (Pin_6)
- net SDO(MISO): now also J6.13 (Pin_13), J6.9 (Pin_9)
- net T_IRQ: now also J6.14 (Pin_14)
- net T_SC: now also J6.11 (Pin_11)

Commit message: connectors
Parts:
- C2: value 1uF tan -> 1uF
- C4: value 10uF tann -> 10uF
Other:
- moved on the sheet: C1, C2, C3, C4, J1, J2, J3, J4, J5, J6

Commit message: PCB
Connections:
- net GND: now also C19.2, D3.2 (A)
- net USB_DM renamed D-
- net USB_DP renamed D+
Changed lines of the file:
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@@
 	)
 	(junction
+		(at 25.4 187.96)
+		(diameter 0)
+		(color 0 0 0 0)
+	)
+	(junction
 		(at 92.71 97.79)
 		(diameter 0)
@@
 	(wire
 		(pts
+			(xy 25.4 187.96) (xy 35.56 187.96)
+		)
+		(stroke
+			(width 0)
+			(type default)
+		)
+	)
+	(wire
+		(pts
 			(xy 25.4 137.16) (xy 27.94 137.16)
 		)
@@
 	(wire
 		(pts
-			(xy 262.89 68.58) (xy 266.7 68.58)
+			(xy 262.89 68.58) (xy 264.16 68.58)
 		)
 		(stroke
@@
 	(wire
 		(pts
-			(xy 15.24 187.96) (xy 35.56 187.96)
-		)
-		(stroke
-			(width 0)
-			(type default)
-		)
-	)
-	(wire
-		(pts
 			(xy 134.62 26.67) (xy 138.43 26.67)
 		)
@@
 	(wire
 		(pts
+			(xy 15.24 187.96) (xy 25.4 187.96)
+		)
+		(stroke
+			(width 0)
+			(type default)
+		)
+	)
+	(wire
+		(pts
 			(xy 17.78 22.86) (xy 19.05 22.86)
 		)
@@
 		)
 	)
+	(wire
+		(pts
+			(xy 25.4 187.96) (xy 25.4 189.23)
+		)
+		(stroke
+			(width 0)
+			(type default)
+		)
+	)
 	(polyline
 		(pts
@@
 	(wire
 		(pts
-			(xy 262.89 66.04) (xy 266.7 66.04)
+			(xy 262.89 66.04) (xy 264.16 66.04)
 		)
 		(stroke
@@
 	(wire
 		(pts
-			(xy 25.4 186.69) (xy 25.4 189.23)
+			(xy 25.4 186.69) (xy 25.4 187.96)
 		)
 		(stroke
@@
 		)
 	)
+	(label "D+"
+		(at 66.04 69.85 0)
+		(effects
+			(font
+				(size 1.27 1.27)
+			)
+			(justify left bottom)
+		)
+	)
+	(label "D+"
+		(at 264.16 68.58 0)
+		(effects
+			(font
+				(size 1.27 1.27)
+			)
+			(justify left bottom)
+		)
+	)
+	(label "D-"
+		(at 66.04 67.31 0)
+		(effects
+			(font
+				(size 1.27 1.27)
+			)
+			(justify left bottom)
+		)
+	)
+	(label "D-"
+		(at 264.16 66.04 0)
+		(effects
+			(font
+				(size 1.27 1.27)
+			)
+			(justify left bottom)
+		)
+	)
 	(global_label "MOSFET_3"
 		(shape input)
@@
 		)
 	)
-	(global_label "USB_DP"
-		(shape input)
-		(at 266.7 68.58 0)
-		(fields_autoplaced yes)
-		(effects
-			(font
-				(size 1.27 1.27)
-			)
-			(justify left)
-		)
-		(property "Intersheetrefs" "${INTERSHEET_REFS}"
-			(at 277.0028 68.58 0)
-			(hide yes)
-			(show_name no)
-			(do_not_autoplace no)
-			(effects
-				(font
-					(size 1.27 1.27)
-				)
-				(justify left)
-			)
-		)
-	)
 	(global_label "TEMP5_MEASURE"
 		(shape input)
@@
 		)
 	)
-	(global_label "USB_DM"
-		(shape input)
-		(at 66.04 67.31 0)
-		(fields_autoplaced yes)
-		(effects
-			(font
-				(size 1.27 1.27)
-			)
-			(justify left)
-		)
-		(property "Intersheetrefs" "${INTERSHEET_REFS}"
-			(at 76.5242 67.31 0)
-			(hide yes)
-			(show_name no)
-			(do_not_autoplace no)
-			(effects
-				(font
-					(size 1.27 1.27)
-				)
-				(justify left)
-			)
-		)
-	)
 	(global_label "DC{slash}RS"
 		(shape input)
@@
 		)
 	)
-	(global_label "USB_DM"
-		(shape input)
-		(at 266.7 66.04 0)
-		(fields_autoplaced yes)
-		(effects
-			(font
-				(size 1.27 1.27)
-			)
-			(justify left)
-		)
-		(property "Intersheetrefs" "${INTERSHEET_REFS}"
-			(at 277.1842 66.04 0)
-			(hide yes)
-			(show_name no)
-			(do_not_autoplace no)
-			(effects
-				(font
-					(size 1.27 1.27)
-				)
-				(justify left)
-			)
-		)
-	)
 	(global_label "SDI(MOSI)"
 		(shape input)
@@
 			)
 		)
-	)
-	(global_label "USB_DP"
-		(shape input)
-		(at 66.04 69.85 0)
-		(fields_autoplaced yes)
-		(effects
-			(font
-				(size 1.27 1.27)
-			)
-			(justify left)
-		)
-		(property "Intersheetrefs" "${INTERSHEET_REFS}"
-			(at 76.3428 69.85 0)
-			(hide yes)
-			(show_name no)
-			(do_not_autoplace no)
-			(effects
-				(font
-					(size 1.27 1.27)
-				)
-				(justify left)
-			)
-		)

Commit message: connectors
Parts:
- removed J4: Conn_01x06_Pin, Connector_PinSocket_2.54mm:PinSocket_1x06_P2.54mm_Vertical, symbol Connector:Conn_01x06_Pin
- removed J5: Conn_01x04_Pin, Connector_PinSocket_2.54mm:PinSocket_1x04_P2.54mm_Vertical, symbol Connector:Conn_01x04_Pin
- added F2, F3, F4, F5: Fuse, Fuse:Fuse_1206_3216Metric_Pad1.42x1.75mm_HandSolder, symbol Device:Fuse
- added J4: Conn_01x04, Connector_JST:JST_EH_B4B-EH-A_1x04_P2.50mm_Vertical, symbol Connector_Generic:Conn_01x04
- added J5: Conn_01x07, Connector_JST:JST_EH_B7B-EH-A_1x07_P2.50mm_Vertical, symbol Connector_Generic:Conn_01x07
- J2: footprint Connector_Samtec_HPM_THT:Samtec_HPM-03-01-x-S_Straight_1x03_Pitch5.08mm -> TerminalBlock:TerminalBlock_MaiXu_MX126-5.0-03P_1x03_P5.00mm
- J3: footprint Connector_PinSocket_2.54mm:PinSocket_1x03_P2.54mm_Vertical -> Connector_PinHeader_2.54mm:PinHeader_1x03_P2.54mm_Vertical
- J6: footprint Connector_PinSocket_2.54mm:PinSocket_2x07_P2.54mm_Vertical -> Connector_JST:JST_PHD_B14B-PHDSS_2x07_P2.00mm_Vertical
Connections:
- net +12V: now also F2.1, F2.2
- net +3.3V: now also J5.6 (Pin_6)
- net DOWN: now also U1.76 (PB7), J5.5 (Pin_5); no longer U1.74 (PB5)
- net GND: now also J5.7 (Pin_7)
- net LEFT: now also J5.4 (Pin_4)
- net LOAD_1: now also F3.1, F3.2, F4.1, F4.2
- net LOAD_2: now also F5.1, F5.2
- net OK: now also U1.74 (PB5), J5.3 (Pin_3); no longer U1.72 (PB3)
- net RIGHT: now also U1.73 (PB4), J5.2 (Pin_2); no longer U1.76 (PB7)
- net SD_CS: now also J4.1 (Pin_1)
- net SD_MISO: now also J4.2 (Pin_2)
- net SD_MOSI: now also J4.3 (Pin_3)
- net SD_SCK: now also J4.4 (Pin_4)
- net UP: now also U1.72 (PB3), J5.1 (Pin_1); no longer U1.73 (PB4)
Other:
- note added: "Fuse"
- moved on the sheet: C3, C4, J1, J6

Commit message: zener diodes
Parts:
- removed D2, D3, D4, D5: BAT46W-E3-08, Diode_SMD:D_SOD-123, symbol Device:D_Schottky
- added D2, D3: D_Zener, Diode_SMD:D_SOD-123F, symbol Device:D_Zener
Connections:
- net GND: now also D2.2 (A), D3.2 (A)
- net V1_MEASURE: now also D2.1 (K)
- net V2_MEASURE: now also D3.1 (K)
