File: untitled.kicad_sch (KiCad schematic)
At the start: 84 parts, among them J10 Conn_01x02, J11 Conn_01x02, J12 Conn_01x02, J13 Conn_01x02, J14 Conn_01x02, J15 Conn_01x02, J16 Conn_01x02, J17 Conn_01x02, J18 Conn_01x02, J19 Conn_01x02, J20 Conn_01x02, J8 Conn_01x02, J9 Conn_01x02, Q1 IXFQ50N60P3, Q10 STP55NF06L, Q11 STP55NF06L, Q2 IXFQ50N60P3, Q3 IXFQ50N60P3, Q4 IXFQ50N60P3, Q5 STP55NF06L, Q6 STP55NF06L, Q7 STP55NF06L, Q8 STP55NF06L, Q9 STP55NF06L, U2 TL074

Commit message: changing the operational amplifier
Parts:
- removed U2: TL074, Package_SO:SO-14_3.9x8.65mm_P1.27mm, symbol Amplifier_Operational:TL074
- added C25, C26, C28: 100n, Capacitor_SMD:C_0805_2012Metric_Pad1.18x1.45mm_HandSolder, symbol Device:C_Small
- added U6, U7, U8, U9: TL071, Package_SO:SO-8_3.9x4.9mm_P1.27mm, symbol Amplifier_Operational:TL071
- J10, J11, J12, J13, J14, J15, J16, J17, J18, J19, J20, J8, J9: footprint (none) -> Connector_PinSocket_2.54mm:PinSocket_1x02_P2.54mm_Vertical
- renumbered C25 to C27, C26 to C29, C27 to C30, C28 to C31, C29 to C32, C30 to C33, C31 to C34
Connections:
- net +12V: now also C25.1, C26.1, C28.1, U6.7 (V+), U7.7 (V+), U8.7 (V+), U9.7 (V+)
- net GND: now also C25.2, C26.2, C28.2, U6.4 (V-), U7.4 (V-), U8.4 (V-), U9.4 (V-)
- net MOSFET1: now also U6.3 (+)
- net MOSFET2: now also U7.3 (+)
- net MOSFET3: now also U8.3 (+)
- net MOSFET4: now also U9.3 (+)
- net at C23.1, R28.1: now also U8.6
- net at C23.2, R29.1: now also U8.2 (-)
- net at C21.1, R12.1: now also U6.6
- net at C22.1, R20.1: now also U7.6
- net at C21.2, R13.1: now also U6.2 (-)
- net at C24.1, R36.1: now also U9.6
- net at C24.2, R37.1: now also U9.2 (-)
- net at C22.2, R21.1: now also U7.2 (-)

Commit message: connectors
Parts:
- removed J17, J18, J19, J20: Conn_01x02, Connector_PinSocket_2.54mm:PinSocket_1x02_P2.54mm_Vertical, symbol Connector_Generic:Conn_01x02
- added J17, J18, J19, J20: Screw_Terminal_01x02, TerminalBlock:TerminalBlock_MaiXu_MX126-5.0-02P_1x02_P5.00mm, symbol Connector:Screw_Terminal_01x02
- J10, J11, J12, J13, J14, J15, J16, J8, J9: footprint Connector_PinSocket_2.54mm:PinSocket_1x02_P2.54mm_Vertical -> Connector_JST:JST_EH_B2B-EH-A_1x02_P2.50mm_Vertical
Connections:
- net LOAD_1: now also J17.1 (Pin_1), J18.1 (Pin_1)
- net LOAD_2: now also J19.1 (Pin_1), J20.1 (Pin_1)
- net at Q8.1 (D): now also J17.2 (Pin_2)
- net at Q9.1 (D): now also J18.2 (Pin_2)
- net at Q10.1 (D): now also J19.2 (Pin_2)
- net at Q11.1 (D): now also J20.2 (Pin_2)

Commit message: zener diodes
Parts:
- renumbered D6 to D4, D7 to D5, D8 to D6
Changed lines of the file:
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@@
 		(in_pos_files yes)
 		(dnp no)
-		(property "Reference" "D6"
+		(property "Reference" "D4"
 			(at 129.794 26.416 90)
 			(show_name no)
@@
 			(project "electronic_load"
 				(path "/eb6f2439-c99a-400f-b3b0-2a7303f23577/2998a9e1-11e1-4086-bdde-6198cb9d05b5"
-					(reference "D6")
+					(reference "D4")
 					(unit 1)
 				)
@@
 		(in_pos_files yes)
 		(dnp no)
-		(property "Reference" "D7"
+		(property "Reference" "D5"
 			(at 129.794 70.866 90)
 			(show_name no)
@@
 			(project "electronic_load"
 				(path "/eb6f2439-c99a-400f-b3b0-2a7303f23577/2998a9e1-11e1-4086-bdde-6198cb9d05b5"
-					(reference "D7")
+					(reference "D5")
 					(unit 1)
 				)
@@
 		(in_pos_files yes)
 		(dnp no)
-		(property "Reference" "D8"
+		(property "Reference" "D6"
 			(at 129.794 117.856 90)
 			(show_name no)
@@
 			(project "electronic_load"
 				(path "/eb6f2439-c99a-400f-b3b0-2a7303f23577/2998a9e1-11e1-4086-bdde-6198cb9d05b5"
-					(reference "D8")
-					(unit 1)
-				)
+					(reference "D6")
+					(unit 1)
+				)
