File: electronic_load.kicad_pcb (KiCad board)
At the start: 2 copper layers, 139 parts, among them J1 Conn_01x02, J10 Conn_01x02, J11 Conn_01x02, J12 Conn_01x02, J13 Conn_01x02, J14 Conn_01x02, J15 Conn_01x02, J16 Conn_01x02, J17 Conn_01x02, J18 Conn_01x02, J19 Conn_01x02, J2 Conn_01x03, J20 Conn_01x02, J3 Conn_01x03_Pin, J4 Conn_01x06_Pin, J5 Conn_01x04_Pin, J6 Conn_01x14_Pin, J7 USB_C_Receptacle_USB2.0_16P, J8 Conn_01x02, J9 Conn_01x02, Q1 IXFQ50N60P3, Q10 STP55NF06L, Q11 STP55NF06L, Q2 IXFQ50N60P3, Q3 IXFQ50N60P3, Q4 IXFQ50N60P3, Q5 STP55NF06L, Q6 STP55NF06L, Q7 STP55NF06L, Q8 STP55NF06L, Q9 STP55NF06L, U1 STM32G491METx, U2 MCP4728, U3 LF33_TO252, U4 NCP1117-5.0_SOT223, U5 USBLC6-2SC6, U6 TL071, U7 TL071, U8 TL071, U9 TL071, Y1 12MHz

Commit message: connectors
Parts:
- C3, C4, R44, R45, R46, R5, R6, R7: moved to B.Cu
- J1: value Conn_01x02 -> Barrel_Jack_Switch_Pin3Ring; footprint Connector_BarrelJack:BarrelJack_Wuerth_694108106102_2.5x5.5mm -> Connector_BarrelJack:BarrelJack_Wuerth_694106106102_2.0x5.5mm
- J10, J11, J12, J13, J14, J15, J16, J8, J9: footprint Connector_PinSocket_2.54mm:PinSocket_1x02_P2.54mm_Vertical -> Connector_JST:JST_EH_B2B-EH-A_1x02_P2.50mm_Vertical
- J17, J18, J19, J20: value Conn_01x02 -> Screw_Terminal_01x02; footprint Connector_PinSocket_2.54mm:PinSocket_1x02_P2.54mm_Vertical -> TerminalBlock:TerminalBlock_MaiXu_MX126-5.0-02P_1x02_P5.00mm
- moved J11 168.0 mm to (38.3, 132.9), turned to 90 degrees
- moved J12 162.4 mm to (38.3, 127.9), turned to 90 degrees
- moved J13 156.9 mm to (38.3, 122.9), turned to 90 degrees
- moved R52 156.2 mm to (47.8, 129.4), turned to 0 degrees
- moved R51 152.1 mm to (47.8, 125.9), turned to 0 degrees
- moved J14 151.5 mm to (38.3, 117.9), turned to 90 degrees
- moved R50 148.1 mm to (47.8, 122.4), turned to 0 degrees
- moved J15 146.3 mm to (38.3, 112.9), turned to 90 degrees
- moved R49 144.1 mm to (47.8, 118.9), turned to 0 degrees
- moved J16 141.7 mm to (38.3, 108.1), turned to 90 degrees
- moved R48 140.2 mm to (47.8, 115.4), turned to 0 degrees
- moved C1 137.9 mm to (72.1, 30.6)
- moved R47 136.3 mm to (47.8, 111.9), turned to 0 degrees
- moved C2 132.2 mm to (77.6, 30.6)
- moved J8 128.2 mm to (45.1, 49.0)
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Connections:
- J1 pad 3: (no net) -> unconnected-(J1-Pad3)
Routing:
- net +12V: track 0.00 -> 58.9 mm
- net SDI(MOSI): track 0.00 -> 39.0 mm
- net Net-(Q4-S): track 0.00 -> 37.9 mm
- net SDO(MISO): track 0.00 -> 34.4 mm, vias 0 -> 1
- net SWDIO: track 0.00 -> 27.5 mm
- net +3.3V: track 0.00 -> 27.1 mm, vias 0 -> 6
- net T_IRQ: track 0.00 -> 25.9 mm
- net DC/RS: track 0.00 -> 23.7 mm
- net SWDCLK: track 0.00 -> 23.6 mm
- net T_SC: track 0.00 -> 23.0 mm
- net SCK: track 0.00 -> 22.3 mm
- net RIGHT: track 0.00 -> 18.4 mm
- net LEFT: track 0.00 -> 16.4 mm
- net MOSFET_4: track 52.7 -> 69.0 mm
- net DOWN: track 0.00 -> 14.4 mm
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
Commit message: connectors
Parts:
- C29, C30, C31, C32, C33, C34, D6, D7, D8, J1, R47, R48, R49, R50, R51, R52, R53, R54, R55, R56: moved to B.Cu
- J6: value Conn_01x14_Pin -> Conn_02x07_Top_Bottom; footprint Connector_PinSocket_2.54mm:PinSocket_1x14_P2.54mm_Vertical -> Connector_PinSocket_2.54mm:PinSocket_2x07_P2.54mm_Vertical
- R44, R45, R46: moved to F.Cu
- moved R52 80.4 mm to (59.4, 49.9)
- moved R51 70.6 mm to (59.2, 56.2), turned to 180 degrees
- moved C34 64.9 mm to (72.0, 49.9), turned to 90 degrees
- moved C33 62.6 mm to (68.6, 49.9), turned to 90 degrees
- moved C32 60.9 mm to (65.3, 49.9), turned to 90 degrees
- moved R50 60.6 mm to (58.8, 62.8), turned to 180 degrees
- moved J16 60.0 mm to (52.3, 49.7), turned to 180 degrees
- moved J15 58.6 mm to (52.3, 56.1), turned to 180 degrees
- moved J14 57.2 mm to (52.3, 62.4), turned to 180 degrees
- moved J13 55.9 mm to (52.2, 68.8), turned to 180 degrees
- moved J12 54.6 mm to (52.2, 75.1), turned to 180 degrees
- moved J11 53.2 mm to (52.3, 81.6), turned to 180 degrees
- moved C31 53.0 mm to (65.4, 55.6), turned to -90 degrees
- moved R49 51.5 mm to (58.9, 68.7), turned to 180 degrees
- moved C30 48.3 mm to (68.7, 55.6), turned to -90 degrees
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Connections:
- U1 pad 17: R1 -> R4
- U1 pad 18: R2 -> R3
- U1 pad 19: R3 -> R2
- U1 pad 20: R4 -> R1
- U1 pad 24: Fan1_PWM -> Fan2_PWM
- U1 pad 25: Fan2_PWM -> Fan1_PWM
- U1 pad 47: CS -> DC/RS
- U1 pad 49: DC/RS -> CS
Routing:
- net R4: track 0.00 -> 99.7 mm
- net R1: track 0.00 -> 98.9 mm
- net R3: track 0.00 -> 90.2 mm
- net R2: track 0.00 -> 89.8 mm
- net Fan3_PWM: track 0.00 -> 65.7 mm, vias 0 -> 1
- net Fan2_PWM: track 0.00 -> 55.0 mm, vias 0 -> 1
- net +12V: track 58.9 -> 6.15 mm
- net Fan1_PWM: track 0.00 -> 43.2 mm, vias 0 -> 1
- net TEMP1_MEASURE: track 0.00 -> 38.6 mm
- net TEMP2_MEASURE: track 0.00 -> 32.2 mm
- net TEMP3_MEASURE: track 0.00 -> 28.4 mm
- net RESET: track 0.00 -> 27.6 mm
- net TEMP4_MEASURE: track 0.00 -> 26.1 mm
- net CS: track 0.00 -> 25.7 mm
- net TEMP5_MEASURE: track 0.00 -> 21.1 mm
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
Commit message: PCB
Parts:
- C2: value 1uF tan -> 1uF
- C4: value 10uF tann -> 10uF
- moved D2 49.0 mm to (86.0, 83.2)
- moved D3 49.0 mm to (86.0, 77.2)
- moved R8 48.9 mm to (90.0, 82.6)
- moved R9 48.9 mm to (90.0, 77.6)
- moved D4 20.5 mm to (86.3, 112.1)
- moved D5 20.5 mm to (86.3, 106.6)
- moved R10 20.5 mm to (90.8, 112.1)
- moved R11 20.5 mm to (90.8, 107.1)
- moved R7 19.3 mm to (90.8, 86.1), turned to 0 degrees
- moved C20 18.7 mm to (74.2, 62.4), turned to 180 degrees
- moved C3 18.6 mm to (96.5, 87.8)
- moved C4 18.4 mm to (96.9, 91.3)
- moved C19 18.3 mm to (75.2, 65.8), turned to 180 degrees
- moved R6 17.5 mm to (90.8, 82.9), turned to 0 degrees
- moved R5 17.5 mm to (90.8, 79.0), turned to 0 degrees
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Connections:
- net USB_DM renamed /D-
- net USB_DP renamed /D+
- C19 pad 2: Net-(D3-A) -> GND
- D3 pad 2: Net-(D3-A) -> GND
Routing:
- net +12V: track 6.15 -> 351.2 mm, vias 0 -> 2
- net LOAD_1: track 0.00 -> 296.6 mm
- net +3.3V: track 35.8 -> 203.2 mm, vias 6 -> 13
- net LOAD_2: track 0.00 -> 126.3 mm
- net V2_MEASURE: track 0.00 -> 73.8 mm, vias 0 -> 3
- net Net-(Q3-S): track 0.00 -> 57.9 mm
- net Net-(Q1-S): track 0.00 -> 56.4 mm
- net Net-(Q2-S): track 0.00 -> 52.4 mm
- net DAC_SCL: track 0.00 -> 47.8 mm, vias 0 -> 2
- net DAC_SDA: track 0.00 -> 46.2 mm, vias 0 -> 2
- net DAC_LDAC: track 0.00 -> 41.5 mm, vias 0 -> 2
- net DAC_RDY: track 0.00 -> 41.2 mm
- net V1_MEASURE: track 0.00 -> 38.2 mm, vias 0 -> 1
- net +5V: track 4.01 -> 35.1 mm
- net VBUS: track 0.00 -> 30.9 mm
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- added copper zone on B.Cu, net GND
- added copper zone on F.Cu, net GND

Commit message: PCB
Parts:
- added REF**: MountingHole_3.2mm_M3, MountingHole:MountingHole_3.2mm_M3, F.Cu at (44.5, 30.7)
- added REF**: MountingHole_3.2mm_M3, MountingHole:MountingHole_3.2mm_M3, F.Cu at (44.5, 168.1)
- added REF**: MountingHole_3.2mm_M3, MountingHole:MountingHole_3.2mm_M3, F.Cu at (123.4, 30.7)
- added REF**: MountingHole_3.2mm_M3, MountingHole:MountingHole_3.2mm_M3, F.Cu at (131.8, 168.4)
- moved J2 5.85 mm to (124.7, 163.6)
- moved J1 4.87 mm to (55.4, 35.6)
- moved C32 3.30 mm to (68.6, 50.0)
- moved C33 3.30 mm to (65.3, 50.0)
- moved J6 2.87 mm to (67.6, 29.7)
- moved C15 1.18 mm to (73.4, 49.0)
- moved C16 1.10 mm to (70.1, 49.0)
Routing:
- net LOAD_2: track 126.3 -> 120.5 mm
- net TEMP5_MEASURE: track 27.2 -> 30.9 mm
- net T_IRQ: track 36.5 -> 33.7 mm
- net SDO(MISO): track 24.7 -> 22.2 mm
- net T_SC: track 16.4 -> 13.8 mm
- net SCK: track 24.0 -> 21.6 mm, vias 1 -> 0
- net TEMP4_MEASURE: track 31.6 -> 34.0 mm
- net SDI(MOSI): track 29.5 -> 31.9 mm
- net +12V: track 351.2 -> 353.2 mm
- net RESET: track 28.2 -> 26.4 mm
- net CS: track 26.3 -> 24.5 mm
- net +3.3V: track 203.2 -> 204.8 mm
- net DC/RS: track 23.4 -> 22.0 mm
- net LOAD_1: track 296.6 -> 296.1 mm

Commit message: connectors
Parts:
- removed REF** (x4): MountingHole_3.2mm_M3, MountingHole:MountingHole_3.2mm_M3
- added F2: Fuse, Fuse:Fuse_1206_3216Metric_Pad1.42x1.75mm_HandSolder, B.Cu at (44.7, 40.4)
- added F3: Fuse, Fuse:Fuse_1206_3216Metric_Pad1.42x1.75mm_HandSolder, F.Cu at (132.1, 162.3)
- added F4: Fuse, Fuse:Fuse_1206_3216Metric_Pad1.42x1.75mm_HandSolder, F.Cu at (106.9, 170.7)
- added F5: Fuse, Fuse:Fuse_1206_3216Metric_Pad1.42x1.75mm_HandSolder, F.Cu at (106.9, 166.9)
- J2: footprint Connector_Samtec_HPM_THT:Samtec_HPM-03-01-x-S_Straight_1x03_Pitch5.08mm -> TerminalBlock:TerminalBlock_MaiXu_MX126-5.0-03P_1x03_P5.00mm
- J3: footprint Connector_PinSocket_2.54mm:PinSocket_1x03_P2.54mm_Vertical -> Connector_PinHeader_2.54mm:PinHeader_1x03_P2.54mm_Vertical
- J4: value Conn_01x06_Pin -> Conn_01x04; footprint Connector_PinSocket_2.54mm:PinSocket_1x06_P2.54mm_Vertical -> Connector_JST:JST_EH_B4B-EH-A_1x04_P2.50mm_Vertical
- J5: value Conn_01x04_Pin -> Conn_01x07; footprint Connector_PinSocket_2.54mm:PinSocket_1x04_P2.54mm_Vertical -> Connector_JST:JST_EH_B7B-EH-A_1x07_P2.50mm_Vertical
- J6: footprint Connector_PinSocket_2.54mm:PinSocket_2x07_P2.54mm_Vertical -> Connector_JST:JST_PHD_B14B-PHDSS_2x07_P2.00mm_Vertical
- moved J4 19.6 mm to (97.9, 54.6), turned to 90 degrees
- moved J5 12.9 mm to (98.6, 61.5), turned to -90 degrees
- moved J6 0.97 mm to (67.1, 30.5), turned to -90 degrees
- moved J2 0.51 mm to (124.7, 163.1), turned to 180 degrees
Connections:
- J4 pad 1: GND -> SD_CS
- J4 pad 2: RIGHT -> SD_MISO
- J4 pad 3: LEFT -> SD_MOSI
- J4 pad 4: DOWN -> SD_SCK
- J5 pad 1: SD_SCK -> UP
- J5 pad 2: SD_MOSI -> RIGHT
- J5 pad 3: SD_MISO -> OK
- J5 pad 4: SD_CS -> LEFT
- U1 pad 72: OK -> UP
- U1 pad 73: UP -> RIGHT
- U1 pad 74: DOWN -> OK
- U1 pad 76: RIGHT -> DOWN
Routing:
- net +3.3V: track 204.8 -> 218.4 mm
- net LOAD_1: track 296.1 -> 287.9 mm
- net RIGHT: track 18.4 -> 12.8 mm
- net LOAD_2: track 120.5 -> 116.0 mm
- net DOWN: track 14.4 -> 18.4 mm
- net OK: track 12.0 -> 14.4 mm
- net SDI(MOSI): track 31.9 -> 30.0 mm
- net T_SC: track 13.8 -> 15.3 mm
- net SD_CS: track 10.4 -> 9.08 mm
- net SD_MOSI: track 10.8 -> 12.0 mm
- net SD_SCK: track 11.8 -> 12.9 mm
- net UP: track 12.8 -> 12.0 mm
- net RESET: track 26.4 -> 25.8 mm
- net GND: vias 468 -> 473

Commit message: zener diodes
Parts:
- removed the D4 at (86.3, 112.1)
- removed the D5 at (86.3, 106.6)
- D2, D3: value BAT46W-E3-08 -> D_Zener; footprint Diode_SMD:D_SOD-123 -> Diode_SMD:D_SOD-123F
- moved D3 29.5 mm to (86.4, 106.7)
- moved D2 6.00 mm to (86.1, 77.2)
- renumbered D6 to D4, D7 to D5, D8 to D6
Connections:
- D2 pad 1: +3.3V -> V1_MEASURE
- D2 pad 2: V1_MEASURE -> GND
- D3 pad 1: V1_MEASURE -> V2_MEASURE
Routing:
- net +3.3V: track 218.4 -> 166.3 mm
- net V2_MEASURE: track 73.8 -> 68.9 mm
- net V1_MEASURE: track 38.2 -> 34.0 mm
- net GND: vias 473 -> 476

Commit message: PCB
Other:
- board outline added: 95.9 x 146 mm

Commit message: mounting hole
Parts:
- added REF**: MountingHole_3.2mm_M3, MountingHole:MountingHole_3.2mm_M3, F.Cu at (43.9, 168.7)
- added REF**: MountingHole_3.2mm_M3, MountingHole:MountingHole_3.2mm_M3, F.Cu at (44.2, 30.7)
- added REF**: MountingHole_3.2mm_M3, MountingHole:MountingHole_3.2mm_M3, F.Cu at (131.8, 168.4)
- added REF**: MountingHole_3.2mm_M3, MountingHole:MountingHole_3.2mm_M3, F.Cu at (123.4, 30.5)
